File: notebook.sch (KiCad schematic (older format))
At the start: 100 parts, among them J1 SWD, J2 BOOT, J3 ConnA, J4 ConnB, Q1 IRF7403, Q2 IRF7403, Q3 IRF7403, Q4 IRF7403, Q5 IRF7403, Q6 IRF7403, Q7 IRF7403, Q8 IRF7403, SW1 RESET, U1 STM32F103ZCT6, U2 IRS2003, U3 IRS2003, U4 PM8834, U5 PM8834, U6 LM2596S-3.3, U7 4050, U8 4050, Y1 16MHz, Y2 32.768kHz

Commit message: WIP schematics
Parts:
- removed C1, C3, C6, C9: 22pF, Capacitor_SMD:C_0402_1005Metric, symbol Device:C_Small
- removed C10, C11, C12, C13: 10uF, Capacitor_SMD:CP_Elec_5x5.4, symbol Device:CP_Small
- removed C14, C15, C16, C17, C7, C8: 100nF, Capacitor_SMD:C_1206_3216Metric, symbol Device:C_Small
- removed C18, C19: 1uF, Capacitor_SMD:C_1206_3216Metric, symbol Device:C_Small
- removed C2: 10nF, Capacitor_SMD:C_0402_1005Metric, symbol Device:C_Small
- removed C20, C21: 100nF, Capacitor_SMD:C_1206_3216Metric, symbol Device:C
- removed C22, C23, C24, C25, C26, C27, C28, C29, C30, C31, C32, C33: 100nF, Capacitor_SMD:C_0402_1005Metric, symbol Device:C_Small
- removed C4, C5: 220uF, Capacitor_SMD:CP_Elec_10x10, symbol Device:CP
- removed D1: SS34, Diode_SMD:D_SMA, symbol Device:D_Small
- removed D10, D11, D4, D5, D6, D7, D8, D9: 1N4148, Diode_SMD:D_SOD-123, symbol Device:D_Small
- removed D2, D3: FR107, Diode_SMD:D_SOD-123, symbol Device:D_Small
- removed H1, H2: VCCin, notebook:MountingHole_4mm_Pad_Thin, symbol Mechanical:MountingHole_Pad
- removed H10: OD4OUT, notebook:MountingHole_4mm_Pad_Thin, symbol Mechanical:MountingHole_Pad
- removed H11: ISOIN1, notebook:MountingHole_4mm_Pad_Thin, symbol Mechanical:MountingHole_Pad
- removed H12: ISOIN2, notebook:MountingHole_4mm_Pad_Thin, symbol Mechanical:MountingHole_Pad
- removed H13: ISOIN3, notebook:MountingHole_4mm_Pad_Thin, symbol Mechanical:MountingHole_Pad
- removed H14: ISOIN4, notebook:MountingHole_4mm_Pad_Thin, symbol Mechanical:MountingHole_Pad
- removed H15: ISOIN5, notebook:MountingHole_4mm_Pad_Thin, symbol Mechanical:MountingHole_Pad
- removed H16: ISOIN6, notebook:MountingHole_4mm_Pad_Thin, symbol Mechanical:MountingHole_Pad
- removed H17: ISOIN7, notebook:MountingHole_4mm_Pad_Thin, symbol Mechanical:MountingHole_Pad
- removed H18: ISOIN8, notebook:MountingHole_4mm_Pad_Thin, symbol Mechanical:MountingHole_Pad
- removed H19: VDDin, notebook:MountingHole_4mm_Pad_Thin, symbol Mechanical:MountingHole_Pad
- removed H20, H21: GND, notebook:MountingHole_4mm_Pad_Thin, symbol Mechanical:MountingHole_Pad
- removed H3: HB1OUT1, notebook:MountingHole_4mm_Pad_Thin, symbol Mechanical:MountingHole_Pad
- removed H4: HB1OUT2, notebook:MountingHole_4mm_Pad_Thin, symbol Mechanical:MountingHole_Pad
- removed H5: HB2OUT1, notebook:MountingHole_4mm_Pad_Thin, symbol Mechanical:MountingHole_Pad
- removed H6: HB2OUT2, notebook:MountingHole_4mm_Pad_Thin, symbol Mechanical:MountingHole_Pad
- removed H7: OD1OUT, notebook:MountingHole_4mm_Pad_Thin, symbol Mechanical:MountingHole_Pad
- removed H8: OD2OUT, notebook:MountingHole_4mm_Pad_Thin, symbol Mechanical:MountingHole_Pad
- removed H9: OD3OUT, notebook:MountingHole_4mm_Pad_Thin, symbol Mechanical:MountingHole_Pad
- removed J1: SWD, Connector_PinSocket_2.54mm:PinSocket_2x03_P2.54mm_Vertical_SMD, symbol Connector_Generic:Conn_02x03_Odd_Even
- removed J2: BOOT, Connector_PinSocket_2.54mm:PinSocket_2x03_P2.54mm_Vertical_SMD, symbol Connector_Generic:Conn_02x03_Odd_Even
- removed J3: ConnA, Connector_PinHeader_2.54mm:PinHeader_2x10_P2.54mm_Vertical_SMD, symbol Connector_Generic:Conn_02x10_Odd_Even
- removed J4: ConnB, Connector_PinHeader_2.54mm:PinHeader_2x10_P2.54mm_Vertical_SMD, symbol Connector_Generic:Conn_02x10_Odd_Even
- removed L1: 33uH, Inductor_SMD:L_12x12mm_H8mm, symbol Device:L
- removed Q1, Q2, Q3, Q4, Q5, Q6, Q7, Q8: IRF7403, Package_SO:SOIC-8_3.9x4.9mm_P1.27mm, symbol Transistor_FET:IRF7403
- removed R1, R2, R3, R4, R5, R6, R7, R8: 22R, Resistor_SMD:R_1206_3216Metric, symbol Device:R_Small
- removed R10, R11, R9: 10K, Resistor_SMD:R_0402_1005Metric, symbol Device:R
- removed SW1: RESET, Button_Switch_SMD:SW_SPST_PTS645, symbol Switch:SW_Push
- removed U1: STM32F103ZCT6, Package_QFP:LQFP-144_20x20mm_P0.5mm, symbol MCU_ST_STM32F1:STM32F103ZCTx
- removed U2, U3: IRS2003, Package_SO:SOIC-8_3.9x4.9mm_P1.27mm, symbol Driver_FET:IRS2003
- removed U4, U5: PM8834, Package_SO:SOIC-8_3.9x4.9mm_P1.27mm, symbol Driver_FET:PM8834
- removed U6: LM2596S-3.3, Package_TO_SOT_SMD:TO-263-5_TabPin3, symbol Regulator_Switching:LM2596S-3.3
- removed U7, U8: 4050, Package_SO:SOIC-16_3.9x9.9mm_P1.27mm, symbol 4xxx:4050
- removed Y1: 16MHz, Crystal:Crystal_SMD_3225-4Pin_3.2x2.5mm, symbol Device:Crystal_GND24
- removed Y2: 32.768kHz, Crystal:Crystal_SMD_3215-2Pin_3.2x1.5mm, symbol Device:Crystal
Connections:
- net labels removed: +3.3V, BOOT0, BOOT1, CA1, CA10, CA11, CA12, CA13, CA14, CA15, CA16, CA17, CA18, CA19, CA2, CA20, CA3, CA4, CA5, CA6, CA7, CA8, CA9, CB1, CB10, CB11, CB12, CB13, CB14, CB15, CB16, CB17, CB18, CB19, CB2, CB20, CB3, CB4, CB5, CB6, CB7, CB8, CB9, GND, HB1IN1, HB1IN2, HB2IN1, HB2IN2, ISOIN1, ISOIN2, ISOIN3, ISOIN4, ISOIN5, ISOIN6, ISOIN7, ISOIN8, NRST, OD1EN, OD1IN, OD2EN, OD2IN, OD3EN, OD3IN, OD4EN, OD4IN, SWCLK, SWDIO, VCC, VDD
- wire segments 501 -> 60
- no-connect marks 5 -> 3
Other:
- note removed: "ADC3_10-12\n"
- note removed: "ADC3_4-8"
- note removed: "TIM1_1/2"
- note removed: "TIM2_3/4"
- note removed: "TIM3_1/2"
- note removed: "TIM4_1/2"
- note removed: "TIM4_3/4"
- note removed: "TIM5_1/2"
- note removed: "TIM8_1/2"
- note removed: "TIM8_3/4"
